Commit message: add navigation with moving obstacles

File: urdf/omni_base.urdf (robot description, URDF)
Before this commit: robot omni_base, 20 links, 19 joints
Joints:
- joint wheel_front_left_joint: limit effort=50.0 velocity=100 -> effort=6.0 velocity=13.123359580052492
- joint wheel_front_right_joint: limit effort=50.0 velocity=100 -> effort=6.0 velocity=13.123359580052492
- joint wheel_rear_left_joint: limit effort=50.0 velocity=100 -> effort=6.0 velocity=13.123359580052492
- joint wheel_rear_right_joint: limit effort=50.0 velocity=100 -> effort=6.0 velocity=13.123359580052492

Commit message: faster velocity and avoid drift update

File: urdf/omni_base.urdf (robot description, URDF)
Before this commit: robot omni_base, 20 links, 19 joints
Links:
- link base_link: mass 34.047 -> 5.0
Joints:
- joint wheel_front_left_joint: limit effort=6.0 velocity=13.123359580052492 -> effort=50.0 velocity=100
- joint wheel_front_right_joint: limit effort=6.0 velocity=13.123359580052492 -> effort=50.0 velocity=100
- joint wheel_rear_left_joint: limit effort=6.0 velocity=13.123359580052492 -> effort=50.0 velocity=100
- joint wheel_rear_right_joint: limit effort=6.0 velocity=13.123359580052492 -> effort=50.0 velocity=100
